Commit message: improve: enhanced code with xacro

File: ackermann_vehicle_description/urdf/mobile_base.xacro (robot description, xacro)
@@ -1,11 +1,13 @@
 <?xml version="1.0"?>
-<robot name="ackermann_vehicle">
+<robot xmlns:xacro="http://www.ros.org/wiki/xacro">
+    <xacro:include filename="$(find ackermann_vehicle_description)/urdf/common_properties.xacro" />
     <link name="base_footprint"/>
     <link name="chassis_link">
-        <inertial>
+        <xacro:box_inertia m="1.875" l="0.347814" w="0.25299" h="0.036" o_xyz="0.0 0.0 0.0" o_rpy="0.0 0.0 0.0"/>
+        <!-- <inertial>
             <origin xyz="0.0 0.0 0.0" rpy="0.0 0.0 0.0"/>
             <mass value="1.875"/>
             <inertia ixx="0.010203115" ixy="0.0" ixz="0.0" iyy="0.019104777" iyz="0.0" izz="0.028902893"/>
-        </inertial>
+        </inertial> -->
         <visual>
             <origin xyz="0.0 0.0 0.0" rpy="0.0 0.0 0.0"/>
